File: plug_controller.kicad_pcb (KiCad board)
At the start: 2 copper layers, 55.9 x 41.9 mm, 20 parts, among them J1 Conn_01x04, J2 Conn_01x01, J3 Conn_01x01, J4 Conn_01x01, J5 Conn_01x01, Q1 MMBT3904L, Q2 MMBT3904L, Q3 MMBT3904L, Q4 MMBT3904L, U1 MOC3063M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

Commit message: add documentation about buying your on SSD
Other:
- net class AC: trace_width 3.69 -> 4
Changed lines of the file:
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@@
     (links 36)
     (no_connects 0)
-    (area 158.774001 72.611 224.865001 121.127143)
+    (area 158.774001 72.611 224.865001 123.209)
     (thickness 1.6)
     (drawings 23)
@@
   (net_class AC ""
     (clearance 1.22)
-    (trace_width 3.69)
+    (trace_width 4)
     (via_dia 1.22)
     (via_drill 0.85)
@@
     (uvia_drill 0.1)
     (add_net "Net-(D1-Pad1)")
+    (add_net "Net-(D1-Pad2)")
     (add_net "Net-(D2-Pad1)")
     (add_net "Net-(F1-Pad1)")
@@
     (uvia_dia 0.3)
     (uvia_drill 0.1)
-    (add_net "Net-(D1-Pad2)")
     (add_net "Net-(D1-Pad3)")
     (add_net "Net-(D2-Pad3)")
